File: Hardware/DA16200_Thing_Plus.brd (EAGLE design)
At the start: 22.9 x 58.4 mm, 114 parts, among them J2 THING_PLUS, J3 Qwiic, J5 USB C, J6 microSD, J7 CORTEX_JTAG_DEBUG_PTH_NS, Q1 20V/4.2A/52mΩ/1.4W, U1 DA16200MOD, U2 CH340E_MSOP10, U3 MCP73831, U5 4MB Flash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

Commit message: Routing
Parts:
- moved R12 0.38 mm to (12.7, 9.65)
- moved R11 0.13 mm to (10.3, 9.65)
Routing:
- net V_USB: track 3.32 -> 56.1 mm
- net EN: track 0.00 -> 19.5 mm
- net N$15: track 0.00 -> 5.40 mm
- net 3.3V: track 11.7 -> 16.1 mm, vias 7 -> 8
- net N$18: track 0.00 -> 2.11 mm
- net N$16: track 0.00 -> 1.08 mm
- net N$13: track 0.00 -> 1.03 mm

Commit message: Routing
Parts:
- added LOGO1: OSHW-LOGOS, SparkFun-Aesthetics:OSHW-LOGO-S
- added LOGO2: SFE_LOGO_NAME_FLAME.1_INCH, SparkFun-Aesthetics:SFE_LOGO_NAME_FLAME_.1
- moved U$64 2.84 mm to (6.73, 9.40)
Routing:
- net V_BATT: track 1.64 -> 32.7 mm, vias 0 -> 2
- net N$24: track 0.00 -> 24.5 mm
- net !RESET!/SPI_CLK: track 32.4 -> 47.7 mm, vias 0 -> 1
- net N$15: track 5.40 -> 15.9 mm, vias 0 -> 2
- net N$19: track 0.00 -> 7.48 mm, vias 0 -> 2
- net N$11: track 0.00 -> 7.21 mm, vias 0 -> 2
- net N$12: track 0.01 -> 6.79 mm, vias 0 -> 2
- net 3.3V: track 16.1 -> 20.9 mm, vias 8 -> 12
- net V_USB: track 56.1 -> 60.2 mm
- net GND: track 1.51 -> 3.27 mm, vias 8 -> 27
- net N$21: track 0.00 -> 1.34 mm
- net N$22: track 3.48 -> 4.24 mm
- net I2C_SCL: track 73.5 -> 72.8 mm
- net I2C_SDA: track 71.7 -> 72.2 mm

Commit message: Buzzard
Parts:
- added U$17: (no value), output:#TXO#0
- added U$29: (no value), output:#RXI#0
- added U$30: (no value), output:#POCI#0
- added U$43: (no value), output:#PICO#0
- added U$46: (no value), output:#SCLK#0
- added U$48: (no value), output:#A2#0
- added U$49: (no value), output:#A3#0
- added U$50: (no value), output:#GND#0
- added U$51: (no value), output:#3V3#0
- added U$52: (no value), output:#VUB#0
- added U$53: (no value), output:#EN#0
- added U$56: (no value), output:THING_PLUS0
- added U$60: (no value), output:#IOC6#0
- added U$71: (no value), output:#WK2#0
- added U$72: (no value), output:#WK1#0
- added U$73: (no value), output:#RTC#0
- added U$74, U$84: (no value), output:#LED#0
- added U$75: (no value), output:#SD#CS##0
- added U$76: (no value), output:##CSB##0
- added U$77: (no value), output:#SCL#0
- added U$78: (no value), output:#SDA#0
- added U$79: (no value), output:#VBT#0
- added U$80, U$81: (no value), output:DA162000
- added U$82: (no value), output:#I�C#0
- added U$83: (no value), output:WP0
- added U$85: (no value), output:#SHLD#0
- added U$86: (no value), output:CHG0
- added U$87: (no value), output:500MA0
- added U$88: (no value), output:100MA0
- added U$89: (no value), output:#CURR#0
- U$28: device output:##RESET##0 -> output:CURR0
- moved LOGO2 23.9 mm to (11.3, 54.4)
- moved U$28 16.7 mm to (8.89, 25.4)
- moved J7 0.76 mm to (7.11, 26.7)

Commit message: Update DA16200_Thing_Plus.brd
Parts:
- removed U$1: (no value), output:#_16#0
- removed U$10: (no value), output:#WS2812_#0
- removed U$11: (no value), output:#0#TX_#0
- removed U$12: (no value), output:#1#RX_#0
- removed U$13: (no value), output:#4#CIPO_#0
- removed U$14: (no value), output:#3#COPI_#0
- removed U$15: (no value), output:#2#SCK_#0
- removed U$18: (no value), output:#29#ADC3_#0
- removed U$19: (no value), output:#28#ADC2_#0
- removed U$2: (no value), output:#_17#0
- removed U$20: (no value), output:#27#ADC1_#0
- removed U$21: (no value), output:#26#ADC0_#0
- removed U$22: (no value), output:#_VUSB#0
- removed U$23: (no value), output:#_EN#0
- removed U$24: (no value), output:#_VBATT#0
- removed U$25: (no value), output:#GND_#0
- removed U$26: (no value), output:#AREF_#0
- removed U$27: (no value), output:#3#3V_#0
- removed U$3: (no value), output:#_18#0
- removed U$32: (no value), SparkFun-Aesthetics:SFE_LOGO_NAME_FLAME_.1
- removed U$33: (no value), output:#SCL_#0
- removed U$34: (no value), output:#SDA_#0
- removed U$36: (no value), output:#_3#3V#0
- removed U$37: (no value), output:#_AREF#0
- removed U$38: (no value), output:#_GND#0
- removed U$39: (no value), output:#_26#ADC0#0
- removed U$4: (no value), output:#_19#0
- removed U$40: (no value), output:#_27#ADC1#0
- removed U$41: (no value), output:#_28#ADC2#0
- removed U$42: (no value), output:#_29#ADC3#0
- removed U$44: (no value), output:THING_PLUS0
- removed U$45: (no value), SparkFun-Aesthetics:SFE_LOGO_NAME_.1
- removed U$47: (no value), output:THING_PLUS_0
- removed U$5: (no value), output:#_20#0
- removed U$54: (no value), output:250
- removed U$55: (no value), output:CHARGE0
- removed U$57: (no value), output:#22_#0
- removed U$58: (no value), output:#21_#0
- removed U$59: (no value), output:#20_#0
- removed U$6: (no value), output:#_21#0
- removed U$61: (no value), output:#19_#0
- removed U$62: (no value), output:#18_#0
- removed U$63: (no value), output:#17_#0
- removed U$65: (no value), output:#16_#0
- removed U$66: (no value), output:#VUSB_#0
- removed U$67: (no value), output:#EN_#0
- removed U$68: (no value), output:#VBATT_#0
- removed U$69, U$70: (no value), output:#_NC#0
- removed U$7: (no value), output:#_22#0
- removed U$8: (no value), output:#_SCL#7#23#0
- removed U$9: (no value), output:#_SDA#6#0
Changed lines of the file:
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@@
 <?xml version="1.0" encoding="utf-8"?>
 <!DOCTYPE eagle SYSTEM "eagle.dtd">
-<eagle version="9.6.2">
+<eagle version="9.5.2">
 <drawing>
 <settings>
@@
 <attribute name="VALUE" value="2.0K" x="10.16" y="26.724" size="0.6096" layer="28" font="vector" ratio="20" rot="MR180" align="top-center"/>
 </element>
-<element name="U$1" library="output" package="#_16#0" value="" x="29.591" y="26.67" smashed="yes"/>
-<element name="U$2" library="output" package="#_17#0" value="" x="29.591" y="29.21" smashed="yes"/>
-<element name="U$3" library="output" package="#_18#0" value="" x="29.591" y="31.75" smashed="yes"/>
-<element name="U$4" library="output" package="#_19#0" value="" x="29.591" y="34.29" smashed="yes"/>
-<element name="U$5" library="output" package="#_20#0" value="" x="29.591" y="36.83" smashed="yes"/>
-<element name="U$6" library="output" package="#_21#0" value="" x="29.591" y="39.37" smashed="yes"/>
-<element name="U$7" library="output" package="#_22#0" value="" x="29.591" y="41.91" smashed="yes"/>
-<element name="U$10" library="output" package="#WS2812_#0" value="" x="45.339" y="49.53" smashed="yes"/>
-<element name="U$11" library="output" package="#0#TX_#0" value="" x="45.339" y="46.99" smashed="yes"/>
-<element name="U$12" library="output" package="#1#RX_#0" value="" x="45.339" y="44.45" smashed="yes"/>
-<element name="U$13" library="output" package="#4#CIPO_#0" value="" x="45.339" y="41.91" smashed="yes"/>
-<element name="U$14" library="output" package="#3#COPI_#0" value="" x="45.339" y="39.37" smashed="yes"/>
-<element name="U$15" library="output" package="#2#SCK_#0" value="" x="45.339" y="36.83" smashed="yes"/>
-<element name="U$8" library="output" package="#_SCL#7#23#0" value="" x="29.591" y="44.45" smashed="yes"/>
-<element name="U$9" library="output" package="#_SDA#6#0" value="" x="29.591" y="46.99" smashed="yes"/>
-<element name="U$18" library="output" package="#29#ADC3_#0" value="" x="45.339" y="31.75" smashed="yes"/>
-<element name="U$19" library="output" package="#28#ADC2_#0" value="" x="45.339" y="29.21" smashed="yes"/>
-<element name="U$20" library="output" package="#27#ADC1_#0" value="" x="45.339" y="26.67" smashed="yes"/>
-<element name="U$21" library="output" package="#26#ADC0_#0" value="" x="45.339" y="24.13" smashed="yes"/>
-<element name="U$22" library="output" package="#_VUSB#0" value="" x="29.591" y="24.13" smashed="yes"/>
-<element name="U$23" library="output" package="#_EN#0" value="" x="29.591" y="21.59" smashed="yes"/>
-<element name="U$24" library="output" package="#_VBATT#0" value="" x="29.591" y="19.05" smashed="yes"/>
-<element name="U$25" library="output" package="#GND_#0" value="" x="45.339" y="21.59" smashed="yes"/>
-<element name="U$26" library="output" package="#AREF_#0" value="" x="45.339" y="19.05" smashed="yes"/>
-<element name="U$27" library="output" package="#3#3V_#0" value="" x="45.339" y="16.51" smashed="yes"/>
 <element name="U$64" library="SparkFun-Aesthetics" package="QWIIC_4MM" value="" x="6.731" y="9.398" smashed="yes" rot="R270"/>
-<element name="U$32" library="SparkFun-Aesthetics" package="SFE_LOGO_NAME_FLAME_.1" value="" x="61.087" y="21.463" smashed="yes" rot="MR0"/>
-<element name="U$54" library="output" package="250" value="" x="53.34" y="15.24" smashed="yes"/>
-<element name="U$55" library="output" package="CHARGE0" value="" x="52.07" y="13.97" smashed="yes"/>
-<element name="U$57" library="output" package="#22_#0" value="" x="29.591" y="41.91" smashed="yes" rot="MR0"/>
-<element name="U$58" library="output" package="#21_#0" value="" x="29.591" y="39.37" smashed="yes" rot="MR0"/>
-<element name="U$59" library="output" package="#20_#0" value="" x="29.591" y="36.83" smashed="yes" rot="MR0"/>
-<element name="U$61" library="output" package="#19_#0" value="" x="29.591" y="34.29" smashed="yes" rot="MR0"/>
-<element name="U$62" library="output" package="#18_#0" value="" x="29.591" y="31.75" smashed="yes" rot="MR0"/>
-<element name="U$63" library="output" package="#17_#0" value="" x="29.591" y="29.21" smashed="yes" rot="MR0"/>
-<element name="U$65" library="output" package="#16_#0" value="" x="29.591" y="26.67" smashed="yes" rot="MR0"/>
-<element name="U$66" library="output" package="#VUSB_#0" value="" x="29.591" y="24.13" smashed="yes" rot="MR0"/>
-<element name="U$67" library="output" package="#EN_#0" value="" x="29.591" y="21.59" smashed="yes" rot="MR0"/>
-<element name="U$68" library="output" package="#VBATT_#0" value="" x="29.591" y="19.05" smashed="yes" rot="MR0"/>
-<element name="U$33" library="output" package="#SCL_#0" value="" x="29.591" y="44.45" smashed="yes" rot="MR0"/>
-<element name="U$34" library="output" package="#SDA_#0" value="" x="29.591" y="46.99" smashed="yes" rot="MR0"/>
 <element name="U$35" library="output" package="#_#RESET##0" value="" x="21.209" y="13.97" smashed="yes" rot="MR0"/>
-<element name="U$36" library="output" package="#_3#3V#0" value="" x="45.339" y="16.51" smashed="yes" rot="MR0"/>
-<element name="U$37" library="output" package="#_AREF#0" value="" x="45.339" y="19.05" smashed="yes" rot="MR0"/>
-<element name="U$38" library="output" package="#_GND#0" value="" x="45.339" y="21.59" smashed="yes" rot="MR0"/>
-<element name="U$39" library="output" package="#_26#ADC0#0" value="" x="45.339" y="24.13" smashed="yes" rot="MR0"/>
-<element name="U$40" library="output" package="#_27#ADC1#0" value="" x="45.339" y="26.67" smashed="yes" rot="MR0"/>
-<element name="U$41" library="output" package="#_28#ADC2#0" value="" x="45.339" y="29.21" smashed="yes" rot="MR0"/>
-<element name="U$42" library="output" package="#_29#ADC3#0" value="" x="45.339" y="31.75" smashed="yes" rot="MR0"/>
-<element name="U$69" library="output" package="#_NC#0" value="" x="45.339" y="34.29" smashed="yes" rot="MR0"/>
-<element name="U$70" library="output" package="#_NC#0" value="" x="45.339" y="34.29" smashed="yes" rot="MR0"/>
 <element name="R8" library="SparkFun-Resistors" package="0402-TIGHT" value="1k" x="21.59" y="6.35" smashed="yes" rot="R270">
 <attribute name="NAME" x="22.152" y="6.35" size="0.6096" layer="25" font="vector" ratio="20" rot="R270" align="bottom-center"/>
@@
 </element>
 <element name="U$16" library="output" package="PWR0" value="" x="19.05" y="5.08" smashed="yes"/>
-<element name="U$45" library="SparkFun-Aesthetics" package="SFE_LOGO_NAME_.1" value="" x="52.451" y="39.0906" smashed="yes"/>
-<element name="U$47" library="output" package="THING_PLUS_0" value="" x="51.943" y="36.195" smashed="yes"/>
-<element name="U$44" library="output" package="THING_PLUS0" value="" x="60.96" y="18.415" smashed="yes" rot="MR0"/>
 <element name="J2" library="SparkFun-Boards" package="THING_PLUS" value="THING_PLUS" x="0" y="0" smashed="yes">
 <attribute name="NAME" x="0" y="-2.54" size="1.27" layer="25" font="vector"/>

Commit message: More buzzard
Parts:
- removed U$28: (no value), output:CURR0
- removed U$35: (no value), output:#_#RESET##0
- removed U$89: (no value), output:#CURR#0
- added U$1: (no value), output:STAT0
- added U$2: (no value), output:CHG0
- added U$3: (no value), output:#CURR#0
- added U$4: (no value), output:#CURR_#0
- added U$5: (no value), output:##RST##0
- moved U$81 0.13 mm to (7.62, 31.6)
Changed lines of the file:
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@@
 <?xml version="1.0" encoding="utf-8"?>
 <!DOCTYPE eagle SYSTEM "eagle.dtd">
-<eagle version="9.5.2">
+<eagle version="9.6.2">
 <drawing>
 <settings>
@@
 </element>
 <element name="U$64" library="SparkFun-Aesthetics" package="QWIIC_4MM" value="" x="6.731" y="9.398" smashed="yes" rot="R270"/>
-<element name="U$35" library="output" package="#_#RESET##0" value="" x="21.209" y="13.97" smashed="yes" rot="MR0"/>
 <element name="R8" library="SparkFun-Resistors" package="0402-TIGHT" value="1k" x="21.59" y="6.35" smashed="yes" rot="R270">
 <attribute name="NAME" x="22.152" y="6.35" size="0.6096" layer="25" font="vector" ratio="20" rot="R270" align="bottom-center"/>
@@
 <element name="U$56" library="output" package="THING_PLUS0" value="" x="15.875" y="34.29" smashed="yes" rot="MR0"/>
 <element name="U$80" library="output" package="DA162000" value="" x="15.24" y="32.639" smashed="yes" rot="MR0"/>
-<element name="U$81" library="output" package="DA162000" value="" x="7.62" y="31.75" smashed="yes"/>
+<element name="U$81" library="output" package="DA162000" value="" x="7.62" y="31.623" smashed="yes"/>
 <element name="U$82" library="output" package="#I�C#0" value="" x="16.383" y="49.784" smashed="yes" rot="MR0"/>
 <element name="U$83" library="output" package="WP0" value="" x="9.017" y="42.926" smashed="yes" rot="MR0"/>
@@
 <element name="U$87" library="output" package="500MA0" value="" x="19.05" y="28.448" smashed="yes" rot="MR0"/>
 <element name="U$88" library="output" package="100MA0" value="" x="18.923" y="26.162" smashed="yes" rot="MR0"/>
-<element name="U$28" library="output" package="CURR0" value="" x="8.89" y="25.4" smashed="yes"/>
-<element name="U$89" library="output" package="#CURR#0" value="" x="18.415" y="23.622" smashed="yes" rot="MR0"/>
+<element name="U$1" library="output" package="STAT0" value="" x="10.287" y="34.29" smashed="yes"/>
+<element name="U$2" library="output" package="CHG0" value="" x="16.51" y="30.48" smashed="yes"/>
+<element name="U$3" library="output" package="#CURR#0" value="" x="8.763" y="25.146" smashed="yes"/>
+<element name="U$4" library="output" package="#CURR_#0" value="" x="18.288" y="23.622" smashed="yes" rot="MR0"/>
+<element name="U$5" library="output" package="##RST##0" value="" x="21.209" y="13.97" smashed="yes" rot="MR0"/>
 </elements>
 <signals>
