File: Hardware/Production/DA16200_Thing_Plus-Panel.brd (EAGLE design)
At the start: 112.3 x 207 mm, 1530 parts, among them J1 Qwiic, J10 CORTEX_JTAG_DEBUG_PTH_NS, J11 Qwiic, J13 USB C, J14 THING_PLUS, J15 CORTEX_JTAG_DEBUG_PTH_NS, J16 Qwiic, J18 USB C, J19 THING_PLUS, J2 THING_PLUS, J20 CORTEX_JTAG_DEBUG_PTH_NS, J21 Qwiic, J23 USB C, J24 THING_PLUS, J25 CORTEX_JTAG_DEBUG_PTH_NS, J26 Qwiic, J28 USB C, J29 THING_PLUS, J3 Qwiic, J30 CORTEX_JTAG_DEBUG_PTH_NS, J31 Qwiic, J33 USB C, J34 THING_PLUS, J35 CORTEX_JTAG_DEBUG_PTH_NS, J36 Qwiic, J38 USB C, J39 THING_PLUS, J40 CORTEX_JTAG_DEBUG_PTH_NS, J41 Qwiic, J43 USB C, J44 THING_PLUS, J45 CORTEX_JTAG_DEBUG_PTH_NS, J46 Qwiic, J48 USB C, J49 THING_PLUS, J5 USB C, J50 CORTEX_JTAG_DEBUG_PTH_NS, J51 Qwiic, J53 USB C, J54 THING_PLUS, J55 CORTEX_JTAG_DEBUG_PTH_NS, J56 Qwiic, J58 USB C, J59 THING_PLUS, J60 CORTEX_JTAG_DEBUG_PTH_NS, J7 CORTEX_JTAG_DEBUG_PTH_NS, J8 USB C, J9 THING_PLUS, Q1 20V/4.2A/52mΩ/1.4W, Q10 20V/4.2A/52mΩ/1.4W, Q11 20V/4.2A/52mΩ/1.4W, Q12 20V/4.2A/52mΩ/1.4W, Q2 20V/4.2A/52mΩ/1.4W, Q3 20V/4.2A/52mΩ/1.4W, Q4 20V/4.2A/52mΩ/1.4W, Q5 20V/4.2A/52mΩ/1.4W, Q6 20V/4.2A/52mΩ/1.4W, Q7 20V/4.2A/52mΩ/1.4W, Q8 20V/4.2A/52mΩ/1.4W, Q9 20V/4.2A/52mΩ/1.4W, U1 DA16200MOD, U10 MCP73831, U11 DA16200MOD, U12 CH340E_MSOP10, U13 XC6222B331MR-G, U14 MCP73831, U15 DA16200MOD, U16 CH340E_MSOP10, U17 XC6222B331MR-G, U18 MCP73831, U19 DA16200MOD, U2 CH340E_MSOP10, U20 CH340E_MSOP10, U21 XC6222B331MR-G, U22 MCP73831, U23 DA16200MOD, U24 CH340E_MSOP10, U25 XC6222B331MR-G, U26 MCP73831, U27 DA16200MOD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

Commit message: Update production files
Parts:
- added C61, C67: 1.0uF, SparkFun-Capacitors:0402-TIGHT
- added C62, C68: 2.2uF, SparkFun-Capacitors:0402-TIGHT
- added C63, C64, C69, C70: 4.7uF, SparkFun-Capacitors:0402-TIGHT
- added C65, C66, C71, C72: 0.1uF, SparkFun-Capacitors:0402-TIGHT
- C11, C2, C36, C41: value 1.0uF -> 0.1uF
- C12, C17, C42, C47: value 2.2uF -> 0.1uF
- C13, C19, C43, C49: value 4.7uF -> 1.0uF
- C14, C38, C4, C44: value 4.7uF -> 2.2uF
- C15, C40, C45, C6: value 0.1uF -> 4.7uF
- C16, C21, C46, C51: value 1.0uF -> 4.7uF
- C18, C23, C24, C29, C48, C53, C54, C59: value 4.7uF -> 0.1uF
- C20, C50: value 0.1uF -> 2.2uF
- C22, C27, C52, C57: value 2.2uF -> 4.7uF
- C25, C55: value 0.1uF -> 1.0uF
- C26, C56: value 1.0uF -> 2.2uF
- C3, C37: value 2.2uF -> 1.0uF
- R105, R123, R13, R141, R159, R177, R195, R213, R33, R51, R69, R87: value 200 -> 10k
- moved C23 98.8 mm to (79.2, 15.7)
- moved C43 96.6 mm to (81.8, 83.7), turned to 90 degrees
- moved C22 94.6 mm to (89.7, 26.2), turned to 270 degrees
- moved C44 93.8 mm to (86.0, 85.3), turned to 180 degrees
- moved C21 92.0 mm to (84.7, 27.7), turned to 180 degrees
- moved C45 91.1 mm to (84.7, 90.4)
- moved C41 81.1 mm to (55.9, 78.5), turned to 180 degrees
- moved C47 80.3 mm to (79.2, 78.5)
- moved C24 79.6 mm to (89.8, 51.4), turned to 90 degrees
- moved C46 79.3 mm to (89.7, 88.9), turned to 270 degrees
- moved C48 64.8 mm to (89.8, 114.2), turned to 90 degrees
- moved C42 60.9 mm to (66.4, 114.2), turned to 90 degrees
- moved C59 58.1 mm to (32.5, 141.2), turned to 180 degrees
- moved C53 53.5 mm to (9.14, 141.2)
- moved C54 53.0 mm to (19.7, 176.9), turned to 90 degrees
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Connections:
- removed net N$107 (its old number): DA_MEAS3.1, U15.15, U15.34, U15.35
- removed net N$117 (its old number): C21.1, D21.C, MEAS4.1, MEAS4.3, Q5.2, R78.2
- removed net N$126 (its old number): R87.1, S9.3
- removed net N$134 (its old number): DA_MEAS4.1, U19.15, U19.34, U19.35
- removed net N$144 (its old number): C26.1, D26.C, MEAS5.1, MEAS5.3, Q6.2, R96.2
- removed net N$153: R105.1, S11.3
- removed net N$161 (its old number): DA_MEAS5.1, U23.15, U23.34, U23.35
- removed net N$171 (its old number): C31.1, D31.C, MEAS6.1, MEAS6.3, Q7.2, R114.2
- removed net N$180 (its old number): R123.1, S13.3
- removed net N$188 (its old number): DA_MEAS6.1, U27.15, U27.34, U27.35
- removed net N$198 (its old number): C36.1, D36.C, MEAS7.1, MEAS7.3, Q8.2, R132.2
- removed net N$215 (its old number): DA_MEAS7.1, U31.15, U31.34, U31.35
- removed net N$225 (its old number): C41.1, D41.C, MEAS8.1, MEAS8.3, Q9.2, R150.2
- removed net N$234 (its old number): R159.1, S17.3
- removed net N$242 (its old number): DA_MEAS8.1, U35.15, U35.34, U35.35
- removed net N$252 (its old number): C46.1, D46.C, MEAS9.1, MEAS9.3, Q10.2, R168.2
- removed net N$261 (its old number): R177.1, S19.3
- removed net N$279 (its old number): C51.1, D51.C, MEAS10.1, MEAS10.3, Q11.2, R186.2
- removed net N$288 (its old number): R195.1, S21.3
- removed net N$296 (its old number): DA_MEAS10.1, U43.15, U43.34, U43.35
- removed net N$306 (its old number): C56.1, D56.C, MEAS11.1, MEAS11.3, Q12.2, R204.2
- removed net N$315: R213.1, S23.3
- removed net N$323: DA_MEAS11.1, U47.15, U47.34, U47.35
- removed net N$36 (its old number): C2.1, D6.C, MEAS1.1, MEAS1.3, Q2.2, R24.2
- removed net N$45 (its old number): R33.1, S3.3
- removed net N$53 (its old number): DA_MEAS1.1, U6.15, U6.34, U6.35
- removed net N$63 (its old number): C11.1, D11.C, MEAS2.1, MEAS2.3, Q3.2, R42.2
- removed net N$72 (its old number): R51.1, S5.3
- removed net N$8 (its old number): R13.1, S2.3
- removed net N$80 (its old number): DA_MEAS2.1, U11.15, U11.34, U11.35
- removed net N$90 (its old number): C16.1, D16.C, MEAS3.1, MEAS3.3, Q4.2, R60.2
- removed net N$99 (its old number): R69.1, S7.3
- new net N$103: C24.1, DA_MEAS3.1, U15.15, U15.34, U15.35
- new net N$113: C25.1, D21.C, MEAS4.1, MEAS4.3, Q5.2, R78.2
- new net N$129: C30.1, DA_MEAS4.1, U19.15, U19.34, U19.35
- new net N$139: C31.1, D26.C, MEAS5.1, MEAS5.3, Q6.2, R96.2
- new net N$155: C36.1, DA_MEAS5.1, U23.15, U23.34, U23.35
- new net N$165: C37.1, D31.C, MEAS6.1, MEAS6.3, Q7.2, R114.2
- new net N$181: C42.1, DA_MEAS6.1, U27.15, U27.34, U27.35
- new net N$191: C43.1, D36.C, MEAS7.1, MEAS7.3, Q8.2, R132.2
- new net N$217: C49.1, D41.C, MEAS8.1, MEAS8.3, Q9.2, R150.2
- new net N$233: C54.1, DA_MEAS8.1, U35.15, U35.34, U35.35
- new net N$243: C55.1, D46.C, MEAS9.1, MEAS9.3, Q10.2, R168.2
- new net N$259: C60.1, DA_MEAS9.1, U39.15, U39.34, U39.35
- new net N$285: C66.1, DA_MEAS10.1, U43.15, U43.34, U43.35
- new net N$295: C67.1, D56.C, MEAS11.1, MEAS11.3, Q12.2, R204.2
- new net N$311: C72.1, DA_MEAS11.1, U47.15, U47.34, U47.35
- new net N$35: C3.1, D6.C, MEAS1.1, MEAS1.3, Q2.2, R24.2
- new net N$51: C12.1, DA_MEAS1.1, U6.15, U6.34, U6.35
- new net N$61: C13.1, D11.C, MEAS2.1, MEAS2.3, Q3.2, R42.2
- new net N$77: C18.1, DA_MEAS2.1, U11.15, U11.34, U11.35
- new net N$87: C19.1, D16.C, MEAS3.1, MEAS3.3, Q4.2, R60.2
- net !RESET!/SPI_CLK: now also R13.1, S2.3; no longer R13.2
- net !RESET!/SPI_CLK1: now also R33.1, S3.3; no longer R33.2
- net !RESET!/SPI_CLK10: now also R195.1, S21.3; no longer R195.2
- net !RESET!/SPI_CLK11: now also R213.1, S23.3; no longer R213.2
- net !RESET!/SPI_CLK2: now also R51.1, S5.3; no longer R51.2
- net !RESET!/SPI_CLK3: now also R69.1, S7.3; no longer R69.2
- net !RESET!/SPI_CLK4: now also R87.1, S9.3; no longer R87.2
- net !RESET!/SPI_CLK5: now also R105.1, S11.3; no longer R105.2
- net !RESET!/SPI_CLK6: now also R123.1, S13.3; no longer R123.2
- net !RESET!/SPI_CLK7: now also R141.1, S15.3; no longer R141.2
- net !RESET!/SPI_CLK8: now also R159.1, S17.3; no longer R159.2
- net !RESET!/SPI_CLK9: now also R177.1, S19.3; no longer R177.2
- net 3.3V: now also R13.2
- net 3.3V1: now also C11.1, C4.1, R33.2; no longer C3.1, C6.1
- net 3.3V10: now also C62.1, C65.1, R195.2; no longer C52.1, C55.1
- net 3.3V11: now also C68.1, C71.1, R213.2; no longer C57.1, C60.1
- net 3.3V2: now also C14.1, C17.1, R51.2; no longer C12.1, C15.1
- net 3.3V3: now also C23.1, R69.2; no longer C17.1
- net 3.3V4: now also C26.1, C29.1, R87.2; no longer C22.1, C25.1
- net 3.3V5: now also C32.1, C35.1, R105.2; no longer C27.1, C30.1
- net 3.3V6: now also C38.1, C41.1, R123.2; no longer C32.1, C35.1
- net 3.3V7: now also C44.1, C47.1, R141.2; no longer C37.1, C40.1
- net 3.3V8: now also C50.1, C53.1, R159.2; no longer C42.1, C45.1
- net 3.3V9: now also C56.1, C59.1, R177.2; no longer C47.1, C50.1
- net GND: now also C2.2
- net GND1: now also C11.2, C12.2; no longer C2.2
- net GND10: now also C61.2, C62.2, C63.2, C64.2, C65.2, C66.2; no longer C51.2, C52.2, C53.2, C54.2, C55.2
- net GND11: now also C67.2, C68.2, C69.2, C70.2, C71.2, C72.2; no longer C56.2, C57.2, C58.2, C59.2, C60.2
- net GND2: now also C16.2, C17.2, C18.2; no longer C11.2, C12.2
- net GND3: now also C21.2, C22.2, C23.2, C24.2; no longer C16.2, C17.2, C18.2
- net GND4: now also C26.2, C27.2, C28.2, C29.2, C30.2; no longer C21.2, C22.2, C23.2, C24.2
- net GND5: now also C31.2, C32.2, C33.2, C34.2, C35.2, C36.2; no longer C26.2, C27.2, C28.2, C29.2, C30.2
- net GND6: now also C37.2, C38.2, C39.2, C40.2, C41.2, C42.2; no longer C31.2, C32.2, C33.2, C34.2, C35.2
- net GND7: now also C43.2, C44.2, C45.2, C46.2, C47.2, C48.2; no longer C36.2, C37.2, C38.2, C39.2, C40.2
- net GND8: now also C49.2, C50.2, C51.2, C52.2, C53.2, C54.2; no longer C41.2, C42.2, C43.2, C44.2, C45.2
- net GND9: now also C55.2, C56.2, C57.2, C58.2, C59.2, C60.2; no longer C46.2, C47.2, C48.2, C49.2, C50.2
- net N$207: now also C48.1, DA_MEAS7.1, U31.15, U31.34, U31.35; no longer R141.1, S15.3
- net N$25: now also C2.1
- net N$269: now also C61.1, D51.C, MEAS10.1, MEAS10.3, Q11.2, R186.2; no longer DA_MEAS9.1, U39.15, U39.34, U39.35
- net V_BATT1: now also C6.1; no longer C5.1
- net V_BATT10: now also C64.1; no longer C54.1
- net V_BATT11: now also C70.1; no longer C59.1
- net V_BATT2: now also C16.1; no longer C14.1
- net V_BATT3: now also C22.1; no longer C19.1
- net V_BATT4: now also C28.1; no longer C24.1
- net V_BATT5: now also C34.1; no longer C29.1
- net V_BATT6: now also C40.1; no longer C34.1
- net V_BATT7: now also C46.1; no longer C39.1
- net V_BATT8: now also C52.1; no longer C44.1
- net V_BATT9: now also C58.1; no longer C49.1
- net V_USB1: now also C5.1; no longer C4.1
- net V_USB10: now also C63.1; no longer C53.1
- net V_USB11: now also C69.1; no longer C58.1
- net V_USB2: now also C15.1; no longer C13.1
- net V_USB3: now also C21.1; no longer C18.1
- net V_USB4: now also C27.1; no longer C23.1
- net V_USB5: now also C33.1; no longer C28.1
- net V_USB6: now also C39.1; no longer C33.1
- net V_USB7: now also C45.1; no longer C38.1
- net V_USB8: now also C51.1; no longer C43.1
- net V_USB9: now also C57.1; no longer C48.1
Routing:
- net N$311: track 0.00 -> 24.0 mm, vias 0 -> 3
- net N$233: track 0.00 -> 24.0 mm, vias 0 -> 3
- net N$285: track 0.00 -> 24.0 mm, vias 0 -> 3
- net N$259: track 0.00 -> 24.0 mm, vias 0 -> 3
- net N$103: track 0.00 -> 24.0 mm, vias 0 -> 3
- net N$77: track 0.00 -> 24.0 mm, vias 0 -> 3
- net N$51: track 0.00 -> 24.0 mm, vias 1 -> 3
- net N$181: track 0.00 -> 24.0 mm, vias 0 -> 3
- net N$129: track 0.00 -> 24.0 mm, vias 0 -> 3
- net N$155: track 0.00 -> 24.0 mm, vias 0 -> 3
- net N$323: track 22.2 -> 0.00 mm, vias 3 -> 0
- net N$296 (its old number): track 22.2 -> 0.00 mm, vias 3 -> 0
- net N$242 (its old number): track 22.2 -> 0.00 mm, vias 3 -> 0
- net N$107 (its old number): track 22.2 -> 0.00 mm, vias 3 -> 0
- net N$80 (its old number): track 22.2 -> 0.00 mm, vias 3 -> 0
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Other:
- board size 112.3 x 207 mm -> 106.7 x 207 mm
- board text added: "v11"
- board text removed: "v10"

Commit message: Update production files
Parts:
- added C73, C74, C80, C81: 4.7uF, SparkFun-Capacitors:0402-TIGHT
- added C75, C76, C77, C82, C83, C84: 0.1uF, SparkFun-Capacitors:0402-TIGHT
- added C78: 1.0uF, SparkFun-Capacitors:0402-TIGHT
- added C79: 2.2uF, SparkFun-Capacitors:0402-TIGHT
- added RST, RST1, RST10, RST11, RST2, RST3, RST4, RST5, RST6, RST7, RST8, RST9: JUMPER-SMT_2_NC_TRACE_SILK, SparkFun-Jumpers:SMT-JUMPER_2_NC_TRACE_SILK
- added U$829: (no value), output:#IOA10#0
- added U$830: (no value), output:#4#TXO#0
- added U$831: (no value), output:#5#RXI#0
- added U$832: (no value), output:#9#POCI#0
- added U$833: (no value), output:#8#PICO#0
- added U$834: (no value), output:#7#SCLK#0
- added U$835: (no value), output:#2#A2#0
- added U$836: (no value), output:#3#A3#0
- added U$837: (no value), output:#DA#0
- added U$838: (no value), output:#MEAS#0
- added U$839: (no value), output:#VBAT#0
- added U$840: (no value), output:##RST##0
- C11, C17, C18, C24, C53, C59, C60, C66: value 0.1uF -> 4.7uF
- C13, C19, C3, C49, C55, C61: value 1.0uF -> 0.1uF
- C14, C20, C26, C56, C62, C68: value 2.2uF -> 0.1uF
- C15, C22, C57, C64: value 4.7uF -> 1.0uF
- C16, C5, C51, C58: value 4.7uF -> 2.2uF
- C21, C27, C28, C33, C34, C40, C63, C69, C70: value 4.7uF -> 0.1uF
- C23, C30, C65, C72: value 0.1uF -> 2.2uF
- C25, C31, C67: value 1.0uF -> 4.7uF
- C29, C36, C71: value 0.1uF -> 1.0uF
- C32, C38: value 2.2uF -> 4.7uF
- C37: value 1.0uF -> 2.2uF
- C4, C50: value 2.2uF -> 1.0uF
- U$100: device output:1000 -> output:5000
- U$101: device output:MA0 -> output:1000
- U$102: device output:SDA0 -> output:MA0
- U$103: device output:SCL0 -> output:SDA0
- U$104: device output:#CSB#0 -> output:SCL0
- U$105: device output:100 -> output:#CSB#0
- U$106: device output:RTC0 -> output:100
- U$107: device output:WK10 -> output:RTC0
- U$108: device output:WK20 -> output:WK10
- U$109: device output:EN0 -> output:WK20
- U$110: device output:VUSB0 -> output:EN0
- U$111: device output:VBAT0 -> output:VUSB0
- U$112: device output:110 -> output:VBAT0
- U$113: device output:#NC#0 -> output:110
- U$114: device output:TX0 -> output:#NC#0
- U$115: device output:RX0 -> output:TX0
- U$116: device output:90 -> output:RX0
- U$117: device output:80 -> output:90
- U$118: device output:70 -> output:80
- U$119: device output:GND0 -> output:70
- U$120: device output:3V30 -> output:GND0
- U$121: device output:#CHG#0 -> output:3V30
- U$122: device output:#CH340#0 -> output:#CHG#0
- U$123: device output:#0#SDA#0 -> output:#CH340#0
- U$124: device output:#1#SCL#0 -> output:#0#SDA#0
- U$125: device output:#6##CSB##0 -> output:#1#SCL#0
- U$126: device output:#11#LED#0 -> output:#6##CSB##0
- U$127: device output:C60 -> output:#11#LED#0
- U$128: device output:#IOA10#0 -> output:C60
- U$129: device output:#4#TXO#0 -> output:#IOA10#0
- U$130: device output:#5#RXI#0 -> output:#4#TXO#0
- U$131: device output:#9#POCI#0 -> output:#5#RXI#0
- U$132: device output:#8#PICO#0 -> output:#9#POCI#0
- U$133: device output:#7#SCLK#0 -> output:#8#PICO#0
- U$134: device output:#2#A2#0 -> output:#7#SCLK#0
- U$135: device output:#3#A3#0 -> output:#2#A2#0
- U$136: device output:#DA#0 -> output:#3#A3#0
- U$137: device output:#MEAS#0 -> output:#DA#0
- U$138: device output:#VBAT#0 -> output:#MEAS#0
- U$139: device SparkFun-Aesthetics:QWIIC_4MM -> output:#VBAT#0
- U$140, U$43: device output:PWR0 -> output:##RST##0
- U$141: device output:#GND#0 -> SparkFun-Aesthetics:QWIIC_4MM
- U$142: device output:#3V3#0 -> output:PWR0
- U$143: device output:#EN#0 -> output:#GND#0
- U$144: device output:#IOC6#0 -> output:#3V3#0
- U$145: device output:#WK2#0 -> output:#EN#0
- U$146: device output:#WK1#0 -> output:#IOC6#0
- U$147: device output:#RTC#0 -> output:#WK2#0
- U$148: device output:THING_PLUS0 -> output:#WK1#0
- U$149, U$219: device output:DA162000 -> output:#RTC#0
- U$150, U$75: device output:DA162000 -> output:THING_PLUS0
- U$151, U$77: device output:#I�C#0 -> output:DA162000
- U$152, U$221: device output:#LED#0 -> output:DA162000
- U$153: device output:#SHLD#0 -> output:#I�C#0
- U$154: device output:STAT0 -> output:#LED#0
- U$155: device output:CHG0 -> output:#SHLD#0
- U$156: device output:##RST##0 -> output:STAT0
- U$157: device output:#MEAS#0 -> output:CHG0
- U$158: device output:#MEAS_#0 -> output:##RST##0
- U$159: device output:G0 -> output:#MEAS#0
- U$160: device output:3V0 -> output:#MEAS_#0
- U$161: device output:IOA7_0 -> output:G0
- U$162: device output:#VU#0 -> output:3V0
- U$163, U$233, U$303, U$373, U$443: device output:#NC#0 -> output:IOA7_0
- U$164, U$234, U$304, U$374, U$94: device output:#NC#0 -> output:#VU#0
- U$168, U$237, U$306, U$375, U$99: device output:5000 -> output:#NC#0
- U$169, U$238, U$307, U$376, U$445: device output:1000 -> output:#NC#0
- U$170: device output:MA0 -> output:5000
- U$171: device output:SDA0 -> output:1000
- U$172: device output:SCL0 -> output:MA0
- U$173: device output:#CSB#0 -> output:SDA0
- U$174: device output:100 -> output:SCL0
- U$175: device output:RTC0 -> output:#CSB#0
- U$176: device output:WK10 -> output:100
- U$177: device output:WK20 -> output:RTC0
- U$178: device output:EN0 -> output:WK10
- U$179: device output:VUSB0 -> output:WK20
- U$180: device output:VBAT0 -> output:EN0
- U$181: device output:110 -> output:VUSB0
- U$182: device output:#NC#0 -> output:VBAT0
- U$183: device output:TX0 -> output:110
- U$184: device output:RX0 -> output:#NC#0
- U$185: device output:90 -> output:TX0
- U$186: device output:80 -> output:RX0
- U$187: device output:70 -> output:90
- U$188: device output:GND0 -> output:80
- U$189: device output:3V30 -> output:70
- U$190: device output:#CHG#0 -> output:GND0
- U$191: device output:#CH340#0 -> output:3V30
- U$192: device output:#0#SDA#0 -> output:#CHG#0
- U$193: device output:#1#SCL#0 -> output:#CH340#0
- U$194: device output:#6##CSB##0 -> output:#0#SDA#0
- U$195: device output:#11#LED#0 -> output:#1#SCL#0
- U$196: device output:C60 -> output:#6##CSB##0
- U$197: device output:#IOA10#0 -> output:#11#LED#0
- U$198: device output:#4#TXO#0 -> output:C60
- U$199: device output:#5#RXI#0 -> output:#IOA10#0
- U$200: device output:#9#POCI#0 -> output:#4#TXO#0
- U$201: device output:#8#PICO#0 -> output:#5#RXI#0
- U$202: device output:#7#SCLK#0 -> output:#9#POCI#0
- U$203: device output:#2#A2#0 -> output:#8#PICO#0
- U$204: device output:#3#A3#0 -> output:#7#SCLK#0
- U$205: device output:#DA#0 -> output:#2#A2#0
- U$206: device output:#MEAS#0 -> output:#3#A3#0
- U$207: device output:#VBAT#0 -> output:#DA#0
- U$208: device SparkFun-Aesthetics:QWIIC_4MM -> output:#MEAS#0
- U$209: device output:PWR0 -> output:#VBAT#0
- U$210: device output:#GND#0 -> output:##RST##0
- U$211: device output:#3V3#0 -> SparkFun-Aesthetics:QWIIC_4MM
- U$212: device output:#EN#0 -> output:PWR0
- U$213: device output:#IOC6#0 -> output:#GND#0
- U$214: device output:#WK2#0 -> output:#3V3#0
- U$215: device output:#WK1#0 -> output:#EN#0
- U$216: device output:#RTC#0 -> output:#IOC6#0
- U$217: device output:THING_PLUS0 -> output:#WK2#0
- U$218, U$288: device output:DA162000 -> output:#WK1#0
- U$220: device output:#I�C#0 -> output:THING_PLUS0
- U$222, U$291: device output:#SHLD#0 -> output:DA162000
- U$223: device output:STAT0 -> output:#I�C#0
- U$224: device output:CHG0 -> output:#LED#0
- U$225: device output:##RST##0 -> output:#SHLD#0
- U$226: device output:#MEAS#0 -> output:STAT0
- U$227: device output:#MEAS_#0 -> output:CHG0
- U$228: device output:G0 -> output:##RST##0
- U$229: device output:3V0 -> output:#MEAS#0
- U$230: device output:IOA7_0 -> output:#MEAS_#0
- U$231: device output:#VU#0 -> output:G0
- U$232, U$302, U$372, U$442, U$512: device output:#NC#0 -> output:3V0
- U$239, U$308, U$377, U$446, U$515: device output:MA0 -> output:#NC#0
- U$240: device output:SDA0 -> output:5000
- U$241: device output:SCL0 -> output:1000
- U$242: device output:#CSB#0 -> output:MA0
- U$243: device output:100 -> output:SDA0
- U$244: device output:RTC0 -> output:SCL0
- U$245: device output:WK10 -> output:#CSB#0
- U$246: device output:WK20 -> output:100
- U$247: device output:EN0 -> output:RTC0
- U$248: device output:VUSB0 -> output:WK10
- U$249: device output:VBAT0 -> output:WK20
- U$250: device output:110 -> output:EN0
- U$251: device output:#NC#0 -> output:VUSB0
- U$252: device output:TX0 -> output:VBAT0
- U$253: device output:RX0 -> output:110
- U$254: device output:90 -> output:#NC#0
- U$255: device output:80 -> output:TX0
- U$256: device output:70 -> output:RX0
- U$257: device output:GND0 -> output:90
- U$258: device output:3V30 -> output:80
- U$259: device output:#CHG#0 -> output:70
- U$260: device output:#CH340#0 -> output:GND0
- U$261: device output:#0#SDA#0 -> output:3V30
- U$262: device output:#1#SCL#0 -> output:#CHG#0
- U$263: device output:#6##CSB##0 -> output:#CH340#0
- U$264: device output:#11#LED#0 -> output:#0#SDA#0
- U$265: device output:C60 -> output:#1#SCL#0
- U$266: device output:#IOA10#0 -> output:#6##CSB##0
- U$267: device output:#4#TXO#0 -> output:#11#LED#0
- U$268: device output:#5#RXI#0 -> output:C60
- U$269: device output:#9#POCI#0 -> output:#IOA10#0
- U$270: device output:#8#PICO#0 -> output:#4#TXO#0
- U$271: device output:#7#SCLK#0 -> output:#5#RXI#0
- U$272: device output:#2#A2#0 -> output:#9#POCI#0
- U$273: device output:#3#A3#0 -> output:#8#PICO#0
- U$274: device output:#DA#0 -> output:#7#SCLK#0
- U$275: device output:#MEAS#0 -> output:#2#A2#0
- U$276: device output:#VBAT#0 -> output:#3#A3#0
- U$277: device SparkFun-Aesthetics:QWIIC_4MM -> output:#DA#0
- U$278: device output:PWR0 -> output:#MEAS#0
- U$279: device output:#GND#0 -> output:#VBAT#0
- U$280: device output:#3V3#0 -> output:##RST##0
- U$281: device output:#EN#0 -> SparkFun-Aesthetics:QWIIC_4MM
- U$282: device output:#IOC6#0 -> output:PWR0
- U$283: device output:#WK2#0 -> output:#GND#0
- U$284: device output:#WK1#0 -> output:#3V3#0
- U$285: device output:#RTC#0 -> output:#EN#0
- U$286: device output:THING_PLUS0 -> output:#IOC6#0
- U$287, U$357: device output:DA162000 -> output:#WK2#0
- U$289: device output:#I�C#0 -> output:#RTC#0
- U$290: device output:#LED#0 -> output:THING_PLUS0
- U$292, U$361: device output:STAT0 -> output:DA162000
- U$293: device output:CHG0 -> output:#I�C#0
- U$294: device output:##RST##0 -> output:#LED#0
- U$295: device output:#MEAS#0 -> output:#SHLD#0
- U$296: device output:#MEAS_#0 -> output:STAT0
- U$297: device output:G0 -> output:CHG0
- U$298: device output:3V0 -> output:##RST##0
- U$299: device output:IOA7_0 -> output:#MEAS#0
- U$300: device output:#VU#0 -> output:#MEAS_#0
- U$301, U$371, U$441, U$511, U$581: device output:#NC#0 -> output:G0
- U$309, U$378, U$447, U$516, U$585: device output:SDA0 -> output:#NC#0
- U$310: device output:SCL0 -> output:5000
- U$311: device output:#CSB#0 -> output:1000
- U$312: device output:100 -> output:MA0
- U$313: device output:RTC0 -> output:SDA0
- U$314: device output:WK10 -> output:SCL0
- U$315: device output:WK20 -> output:#CSB#0
- U$316: device output:EN0 -> output:100
- U$317: device output:VUSB0 -> output:RTC0
- U$318: device output:VBAT0 -> output:WK10
- U$319: device output:110 -> output:WK20
- U$320: device output:#NC#0 -> output:EN0
- U$321: device output:TX0 -> output:VUSB0
- U$322: device output:RX0 -> output:VBAT0
- U$323: device output:90 -> output:110
- U$324: device output:80 -> output:#NC#0
- U$325: device output:70 -> output:TX0
- U$326: device output:GND0 -> output:RX0
- U$327: device output:3V30 -> output:90
- U$328: device output:#CHG#0 -> output:80
- U$329: device output:#CH340#0 -> output:70
- U$330: device output:#0#SDA#0 -> output:GND0
- U$331: device output:#1#SCL#0 -> output:3V30
- U$332: device output:#6##CSB##0 -> output:#CHG#0
- U$333: device output:#11#LED#0 -> output:#CH340#0
- U$334: device output:C60 -> output:#0#SDA#0
- U$335: device output:#IOA10#0 -> output:#1#SCL#0
- U$336: device output:#4#TXO#0 -> output:#6##CSB##0
- U$337: device output:#5#RXI#0 -> output:#11#LED#0
- U$338: device output:#9#POCI#0 -> output:C60
- U$339: device output:#8#PICO#0 -> output:#IOA10#0
- U$340: device output:#7#SCLK#0 -> output:#4#TXO#0
- U$341: device output:#2#A2#0 -> output:#5#RXI#0
- U$342: device output:#3#A3#0 -> output:#9#POCI#0
- U$343: device output:#DA#0 -> output:#8#PICO#0
- U$344: device output:#MEAS#0 -> output:#7#SCLK#0
- U$345: device output:#VBAT#0 -> output:#2#A2#0
- U$346: device SparkFun-Aesthetics:QWIIC_4MM -> output:#3#A3#0
- U$347: device output:PWR0 -> output:#DA#0
- U$348: device output:#GND#0 -> output:#MEAS#0
- U$349: device output:#3V3#0 -> output:#VBAT#0
- U$350: device output:#EN#0 -> output:##RST##0
- U$351: device output:#IOC6#0 -> SparkFun-Aesthetics:QWIIC_4MM
- U$352: device output:#WK2#0 -> output:PWR0
- U$353: device output:#WK1#0 -> output:#GND#0
- U$354: device output:#RTC#0 -> output:#3V3#0
- U$355: device output:THING_PLUS0 -> output:#EN#0
- U$356, U$426: device output:DA162000 -> output:#IOC6#0
- U$358: device output:#I�C#0 -> output:#WK1#0
- U$359: device output:#LED#0 -> output:#RTC#0
- U$360: device output:#SHLD#0 -> output:THING_PLUS0
- U$362, U$431: device output:CHG0 -> output:DA162000
- U$363: device output:##RST##0 -> output:#I�C#0
- U$364: device output:#MEAS#0 -> output:#LED#0
- U$365: device output:#MEAS_#0 -> output:#SHLD#0
- U$366: device output:G0 -> output:STAT0
- U$367: device output:3V0 -> output:CHG0
- U$368: device output:IOA7_0 -> output:##RST##0
- U$369: device output:#VU#0 -> output:#MEAS#0
- U$370, U$440, U$510, U$580, U$650: device output:#NC#0 -> output:#MEAS_#0
- U$379, U$448, U$517, U$586, U$655: device output:SCL0 -> output:#NC#0
- U$380: device output:#CSB#0 -> output:5000
- U$381: device output:100 -> output:1000
- U$382: device output:RTC0 -> output:MA0
- U$383: device output:WK10 -> output:SDA0
- U$384: device output:WK20 -> output:SCL0
- U$385: device output:EN0 -> output:#CSB#0
- U$386: device output:VUSB0 -> output:100
- U$387: device output:VBAT0 -> output:RTC0
- U$388: device output:110 -> output:WK10
- U$389: device output:#NC#0 -> output:WK20
- U$390: device output:TX0 -> output:EN0
- U$391: device output:RX0 -> output:VUSB0
- U$392: device output:90 -> output:VBAT0
- U$393: device output:80 -> output:110
- U$394: device output:70 -> output:#NC#0
- U$395: device output:GND0 -> output:TX0
- U$396: device output:3V30 -> output:RX0
- U$397: device output:#CHG#0 -> output:90
- U$398: device output:#CH340#0 -> output:80
- U$399: device output:#0#SDA#0 -> output:70
- U$400: device output:#1#SCL#0 -> output:GND0
- U$401: device output:#6##CSB##0 -> output:3V30
- U$402: device output:#11#LED#0 -> output:#CHG#0
- U$403: device output:C60 -> output:#CH340#0
- U$404: device output:#IOA10#0 -> output:#0#SDA#0
- U$405: device output:#4#TXO#0 -> output:#1#SCL#0
- U$406: device output:#5#RXI#0 -> output:#6##CSB##0
- U$407: device output:#9#POCI#0 -> output:#11#LED#0
- U$408: device output:#8#PICO#0 -> output:C60
- U$409: device output:#7#SCLK#0 -> output:#IOA10#0
- U$410: device output:#2#A2#0 -> output:#4#TXO#0
- U$411: device output:#3#A3#0 -> output:#5#RXI#0
- U$412: device output:#DA#0 -> output:#9#POCI#0
- U$413: device output:#MEAS#0 -> output:#8#PICO#0
- U$414: device output:#VBAT#0 -> output:#7#SCLK#0
- U$415: device SparkFun-Aesthetics:QWIIC_4MM -> output:#2#A2#0
- U$416: device output:PWR0 -> output:#3#A3#0
- U$417: device output:#GND#0 -> output:#DA#0
- U$418: device output:#3V3#0 -> output:#MEAS#0
- U$419: device output:#EN#0 -> output:#VBAT#0
- U$420: device output:#IOC6#0 -> output:##RST##0
- U$421: device output:#WK2#0 -> SparkFun-Aesthetics:QWIIC_4MM
- U$422: device output:#WK1#0 -> output:PWR0
- U$423: device output:#RTC#0 -> output:#GND#0
- U$424: device output:THING_PLUS0 -> output:#3V3#0
- U$425, U$495: device output:DA162000 -> output:#EN#0
- U$427: device output:#I�C#0 -> output:#WK2#0
- U$428: device output:#LED#0 -> output:#WK1#0
- U$429: device output:#SHLD#0 -> output:#RTC#0
- U$430: device output:STAT0 -> output:THING_PLUS0
- U$432, U$501: device output:##RST##0 -> output:DA162000
- U$433: device output:#MEAS#0 -> output:#I�C#0
- U$434: device output:#MEAS_#0 -> output:#LED#0
- U$435: device output:G0 -> output:#SHLD#0
- U$436: device output:3V0 -> output:STAT0
- U$437: device output:IOA7_0 -> output:CHG0
- U$438: device output:#VU#0 -> output:##RST##0
- U$439, U$509, U$579, U$649, U$719: device output:#NC#0 -> output:#MEAS#0
- U$444: device output:5000 -> output:#VU#0
- U$449, U$518, U$587, U$656, U$725: device output:#CSB#0 -> output:#NC#0
- U$450: device output:100 -> output:5000
- U$451: device output:RTC0 -> output:1000
- U$452: device output:WK10 -> output:MA0
- U$453: device output:WK20 -> output:SDA0
- U$454: device output:EN0 -> output:SCL0
- U$455: device output:VUSB0 -> output:#CSB#0
- U$456: device output:VBAT0 -> output:100
- U$457: device output:110 -> output:RTC0
- U$458: device output:#NC#0 -> output:WK10
- U$459: device output:TX0 -> output:WK20
- U$46: device output:#GND#0 -> output:PWR0
- U$460: device output:RX0 -> output:EN0
- U$461: device output:90 -> output:VUSB0
- U$462: device output:80 -> output:VBAT0
- U$463: device output:70 -> output:110
- U$464: device output:GND0 -> output:#NC#0
- U$465: device output:3V30 -> output:TX0
- U$466: device output:#CHG#0 -> output:RX0
- U$467: device output:#CH340#0 -> output:90
- U$468: device output:#0#SDA#0 -> output:80
- U$469: device output:#1#SCL#0 -> output:70
- U$470: device output:#6##CSB##0 -> output:GND0
- U$471: device output:#11#LED#0 -> output:3V30
- U$472: device output:C60 -> output:#CHG#0
- U$473: device output:#IOA10#0 -> output:#CH340#0
- U$474: device output:#4#TXO#0 -> output:#0#SDA#0
- U$475: device output:#5#RXI#0 -> output:#1#SCL#0
- U$476: device output:#9#POCI#0 -> output:#6##CSB##0
- U$477: device output:#8#PICO#0 -> output:#11#LED#0
- U$478: device output:#7#SCLK#0 -> output:C60
- U$479: device output:#2#A2#0 -> output:#IOA10#0
- U$48: device output:#3V3#0 -> output:#GND#0
- U$480: device output:#3#A3#0 -> output:#4#TXO#0
- U$481: device output:#DA#0 -> output:#5#RXI#0
- U$482: device output:#MEAS#0 -> output:#9#POCI#0
- U$483: device output:#VBAT#0 -> output:#8#PICO#0
- U$484: device SparkFun-Aesthetics:QWIIC_4MM -> output:#7#SCLK#0
- U$485: device output:PWR0 -> output:#2#A2#0
- U$486: device output:#GND#0 -> output:#3#A3#0
- U$487: device output:#3V3#0 -> output:#DA#0
- U$488: device output:#EN#0 -> output:#MEAS#0
- U$489: device output:#IOC6#0 -> output:#VBAT#0
- U$49: device output:#EN#0 -> output:#3V3#0
- U$490: device output:#WK2#0 -> output:##RST##0
- U$491: device output:#WK1#0 -> SparkFun-Aesthetics:QWIIC_4MM
- U$492: device output:#RTC#0 -> output:PWR0
- U$493: device output:THING_PLUS0 -> output:#GND#0
- U$494, U$564: device output:DA162000 -> output:#3V3#0
- U$496: device output:#I�C#0 -> output:#IOC6#0
- U$497: device output:#LED#0 -> output:#WK2#0
- U$498: device output:#SHLD#0 -> output:#WK1#0
- U$499: device output:STAT0 -> output:#RTC#0
- U$500: device output:CHG0 -> output:THING_PLUS0
- U$502, U$571: device output:#MEAS#0 -> output:DA162000
- U$503: device output:#MEAS_#0 -> output:#I�C#0
- U$504: device output:G0 -> output:#LED#0
- U$505: device output:3V0 -> output:#SHLD#0
- U$506: device output:IOA7_0 -> output:STAT0
- U$507: device output:#VU#0 -> output:CHG0
- U$508, U$578, U$648, U$718, U$788: device output:#NC#0 -> output:##RST##0
- U$513: device output:5000 -> output:IOA7_0
- U$514: device output:1000 -> output:#VU#0
- U$519, U$588, U$657, U$726, U$795: device output:100 -> output:#NC#0
- U$52: device output:#IOC6#0 -> output:#EN#0
- U$520: device output:RTC0 -> output:5000
- U$521: device output:WK10 -> output:1000
- U$522: device output:WK20 -> output:MA0
- U$523: device output:EN0 -> output:SDA0
- U$524: device output:VUSB0 -> output:SCL0
- U$525: device output:VBAT0 -> output:#CSB#0
- U$526: device output:110 -> output:100
- U$527: device output:#NC#0 -> output:RTC0
- U$528: device output:TX0 -> output:WK10
- U$529: device output:RX0 -> output:WK20
- U$530: device output:90 -> output:EN0
- U$531: device output:80 -> output:VUSB0
- U$532: device output:70 -> output:VBAT0
- U$533: device output:GND0 -> output:110
- U$534: device output:3V30 -> output:#NC#0
- U$535: device output:#CHG#0 -> output:TX0
- U$536: device output:#CH340#0 -> output:RX0
- U$537: device output:#0#SDA#0 -> output:90
- U$538: device output:#1#SCL#0 -> output:80
- U$539: device output:#6##CSB##0 -> output:70
- U$54: device output:#WK2#0 -> output:#IOC6#0
- U$540: device output:#11#LED#0 -> output:GND0
- U$541: device output:C60 -> output:3V30
- U$542: device output:#IOA10#0 -> output:#CHG#0
- U$543: device output:#4#TXO#0 -> output:#CH340#0
- U$544: device output:#5#RXI#0 -> output:#0#SDA#0
- U$545: device output:#9#POCI#0 -> output:#1#SCL#0
- U$546: device output:#8#PICO#0 -> output:#6##CSB##0
- U$547: device output:#7#SCLK#0 -> output:#11#LED#0
- U$548: device output:#2#A2#0 -> output:C60
- U$549: device output:#3#A3#0 -> output:#IOA10#0
- U$550: device output:#DA#0 -> output:#4#TXO#0
- U$551: device output:#MEAS#0 -> output:#5#RXI#0
- U$552: device output:#VBAT#0 -> output:#9#POCI#0
- U$553: device SparkFun-Aesthetics:QWIIC_4MM -> output:#8#PICO#0
- U$554: device output:PWR0 -> output:#7#SCLK#0
- U$555: device output:#GND#0 -> output:#2#A2#0
- U$556: device output:#3V3#0 -> output:#3#A3#0
- U$557: device output:#EN#0 -> output:#DA#0
- U$558: device output:#IOC6#0 -> output:#MEAS#0
- U$559: device output:#WK2#0 -> output:#VBAT#0
- U$560: device output:#WK1#0 -> output:##RST##0
- U$561: device output:#RTC#0 -> SparkFun-Aesthetics:QWIIC_4MM
- U$562: device output:THING_PLUS0 -> output:PWR0
- U$563, U$633: device output:DA162000 -> output:#GND#0
- U$565: device output:#I�C#0 -> output:#EN#0
- U$566: device output:#LED#0 -> output:#IOC6#0
- U$567: device output:#SHLD#0 -> output:#WK2#0
- U$568: device output:STAT0 -> output:#WK1#0
- U$569: device output:CHG0 -> output:#RTC#0
- U$570: device output:##RST##0 -> output:THING_PLUS0
- U$572, U$641: device output:#MEAS_#0 -> output:DA162000
- U$573: device output:G0 -> output:#I�C#0
- U$574: device output:3V0 -> output:#LED#0
- U$575: device output:IOA7_0 -> output:#SHLD#0
- U$576: device output:#VU#0 -> output:STAT0
- U$577, U$647, U$717, U$787: device output:#NC#0 -> output:CHG0
- U$58: device output:#WK1#0 -> output:#WK2#0
- U$582: device output:5000 -> output:3V0
- U$583: device output:1000 -> output:IOA7_0
- U$584: device output:MA0 -> output:#VU#0
- U$589, U$658, U$727, U$796: device output:RTC0 -> output:#NC#0
- U$590: device output:WK10 -> output:5000
- U$591: device output:WK20 -> output:1000
- U$592: device output:EN0 -> output:MA0
- U$593: device output:VUSB0 -> output:SDA0
- U$594: device output:VBAT0 -> output:SCL0
- U$595: device output:110 -> output:#CSB#0
- U$596: device output:#NC#0 -> output:100
- U$597: device output:TX0 -> output:RTC0
- U$598: device output:RX0 -> output:WK10
- U$599: device output:90 -> output:WK20
- U$600: device output:80 -> output:EN0
- U$601: device output:70 -> output:VUSB0
- U$602: device output:GND0 -> output:VBAT0
- U$603: device output:3V30 -> output:110
- U$604: device output:#CHG#0 -> output:#NC#0
- U$605: device output:#CH340#0 -> output:TX0
- U$606: device output:#0#SDA#0 -> output:RX0
- U$607: device output:#1#SCL#0 -> output:90
- U$608: device output:#6##CSB##0 -> output:80
- U$609: device output:#11#LED#0 -> output:70
- U$61: device output:#RTC#0 -> output:#WK1#0
- U$610: device output:C60 -> output:GND0
- U$611: device output:#IOA10#0 -> output:3V30
- U$612: device output:#4#TXO#0 -> output:#CHG#0
- U$613: device output:#5#RXI#0 -> output:#CH340#0
- U$614: device output:#9#POCI#0 -> output:#0#SDA#0
- U$615: device output:#8#PICO#0 -> output:#1#SCL#0
- U$616: device output:#7#SCLK#0 -> output:#6##CSB##0
- U$617: device output:#2#A2#0 -> output:#11#LED#0
- U$618: device output:#3#A3#0 -> output:C60
- U$619: device output:#DA#0 -> output:#IOA10#0
- U$620: device output:#MEAS#0 -> output:#4#TXO#0
- U$621: device output:#VBAT#0 -> output:#5#RXI#0
- U$622: device SparkFun-Aesthetics:QWIIC_4MM -> output:#9#POCI#0
- U$623: device output:PWR0 -> output:#8#PICO#0
- U$624: device output:#GND#0 -> output:#7#SCLK#0
- U$625: device output:#3V3#0 -> output:#2#A2#0
- U$626: device output:#EN#0 -> output:#3#A3#0
- U$627: device output:#IOC6#0 -> output:#DA#0
- U$628: device output:#WK2#0 -> output:#MEAS#0
- U$629: device output:#WK1#0 -> output:#VBAT#0
- U$630: device output:#RTC#0 -> output:##RST##0
- U$631: device output:THING_PLUS0 -> SparkFun-Aesthetics:QWIIC_4MM
- U$632, U$702: device output:DA162000 -> output:PWR0
- U$634: device output:#I�C#0 -> output:#3V3#0
- U$635: device output:#LED#0 -> output:#EN#0
- U$636: device output:#SHLD#0 -> output:#IOC6#0
- U$637: device output:STAT0 -> output:#WK2#0
- U$638: device output:CHG0 -> output:#WK1#0
- U$639: device output:##RST##0 -> output:#RTC#0
- U$640: device output:#MEAS#0 -> output:THING_PLUS0
- U$642, U$711: device output:G0 -> output:DA162000
- U$643: device output:3V0 -> output:#I�C#0
- U$644: device output:IOA7_0 -> output:#LED#0
- U$645: device output:#VU#0 -> output:#SHLD#0
- U$646, U$716, U$786: device output:#NC#0 -> output:STAT0
- U$651: device output:5000 -> output:G0
- U$652: device output:1000 -> output:3V0
- U$653: device output:MA0 -> output:IOA7_0
- U$654: device output:SDA0 -> output:#VU#0
- U$659, U$728, U$797: device output:WK10 -> output:#NC#0
- U$660: device output:WK20 -> output:5000
- U$661: device output:EN0 -> output:1000
- U$662: device output:VUSB0 -> output:MA0
- U$663: device output:VBAT0 -> output:SDA0
- U$664: device output:110 -> output:SCL0
- U$665: device output:#NC#0 -> output:#CSB#0
- U$666: device output:TX0 -> output:100
- U$667: device output:RX0 -> output:RTC0
- U$668: device output:90 -> output:WK10
- U$669: device output:80 -> output:WK20
- U$670: device output:70 -> output:EN0
- U$671: device output:GND0 -> output:VUSB0
- U$672: device output:3V30 -> output:VBAT0
- U$673: device output:#CHG#0 -> output:110
- U$674: device output:#CH340#0 -> output:#NC#0
- U$675: device output:#0#SDA#0 -> output:TX0
- U$676: device output:#1#SCL#0 -> output:RX0
- U$677: device output:#6##CSB##0 -> output:90
- U$678: device output:#11#LED#0 -> output:80
- U$679: device output:C60 -> output:70
- U$680: device output:#IOA10#0 -> output:GND0
- U$681: device output:#4#TXO#0 -> output:3V30
- U$682: device output:#5#RXI#0 -> output:#CHG#0
- U$683: device output:#9#POCI#0 -> output:#CH340#0
- U$684: device output:#8#PICO#0 -> output:#0#SDA#0
- U$685: device output:#7#SCLK#0 -> output:#1#SCL#0
- U$686: device output:#2#A2#0 -> output:#6##CSB##0
- U$687: device output:#3#A3#0 -> output:#11#LED#0
- U$688: device output:#DA#0 -> output:C60
- U$689: device output:#MEAS#0 -> output:#IOA10#0
- U$690: device output:#VBAT#0 -> output:#4#TXO#0
- U$691: device SparkFun-Aesthetics:QWIIC_4MM -> output:#5#RXI#0
- U$692: device output:PWR0 -> output:#9#POCI#0
- U$693: device output:#GND#0 -> output:#8#PICO#0
- U$694: device output:#3V3#0 -> output:#7#SCLK#0
- U$695: device output:#EN#0 -> output:#2#A2#0
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Connections:
- removed net N$103 (its old number): C24.1, DA_MEAS3.1, U15.15, U15.34, U15.35
- removed net N$129 (its old number): C30.1, DA_MEAS4.1, U19.15, U19.34, U19.35
- removed net N$155 (its old number): C36.1, DA_MEAS5.1, U23.15, U23.34, U23.35
- removed net N$181 (its old number): C42.1, DA_MEAS6.1, U27.15, U27.34, U27.35
- removed net N$207 (its old number): C48.1, DA_MEAS7.1, U31.15, U31.34, U31.35
- removed net N$233 (its old number): C54.1, DA_MEAS8.1, U35.15, U35.34, U35.35
- removed net N$25 (its old number): C2.1, DA_MEAS.1, U1.15, U1.34, U1.35
- removed net N$259 (its old number): C60.1, DA_MEAS9.1, U39.15, U39.34, U39.35
- removed net N$285 (its old number): C66.1, DA_MEAS10.1, U43.15, U43.34, U43.35
- removed net N$311 (its old number): C72.1, DA_MEAS11.1, U47.15, U47.34, U47.35
- removed net N$51 (its old number): C12.1, DA_MEAS1.1, U6.15, U6.34, U6.35
- removed net N$77 (its old number): C18.1, DA_MEAS2.1, U11.15, U11.34, U11.35
- new net !RESET!: J2.28, R13.1, RST.1, S2.3
- new net !RESET!1: J9.28, R33.1, RST1.1, S3.3
- new net !RESET!10: J54.28, R195.1, RST10.1, S21.3
- new net !RESET!11: J59.28, R213.1, RST11.1, S23.3
- new net !RESET!2: J14.28, R51.1, RST2.1, S5.3
- new net !RESET!3: J19.28, R69.1, RST3.1, S7.3
- new net !RESET!4: J24.28, R87.1, RST4.1, S9.3
- new net !RESET!5: J29.28, R105.1, RST5.1, S11.3
- new net !RESET!6: J34.28, R123.1, RST6.1, S13.3
- new net !RESET!7: J39.28, R141.1, RST7.1, S15.3
- new net !RESET!8: J44.28, R159.1, RST8.1, S17.3
- new net !RESET!9: J49.28, R177.1, RST9.1, S19.3
- new net N$104: C27.1, C28.1, DA_MEAS3.1, U15.15, U15.34, U15.35
- new net N$130: C34.1, C35.1, DA_MEAS4.1, U19.15, U19.34, U19.35
- new net N$156: C41.1, C42.1, DA_MEAS5.1, U23.15, U23.34, U23.35
- new net N$182: C48.1, C49.1, DA_MEAS6.1, U27.15, U27.34, U27.35
- new net N$208: C55.1, C56.1, DA_MEAS7.1, U31.15, U31.34, U31.35
- new net N$234: C62.1, C63.1, DA_MEAS8.1, U35.15, U35.34, U35.35
- new net N$260: C69.1, C70.1, DA_MEAS9.1, U39.15, U39.34, U39.35
- new net N$286: C76.1, C77.1, DA_MEAS10.1, U43.15, U43.34, U43.35
- new net N$312: C83.1, C84.1, DA_MEAS11.1, U47.15, U47.34, U47.35
- new net N$52: C13.1, C14.1, DA_MEAS1.1, U6.15, U6.34, U6.35
- new net N$78: C20.1, C21.1, DA_MEAS2.1, U11.15, U11.34, U11.35
- new net N$8: C2.1, C3.1, DA_MEAS.1, U1.15, U1.34, U1.35
- net !RESET!/SPI_CLK: now also RST.2; no longer J2.28, R13.1, S2.3
- net !RESET!/SPI_CLK1: now also RST1.2; no longer J9.28, R33.1, S3.3
- net !RESET!/SPI_CLK10: now also RST10.2; no longer J54.28, R195.1, S21.3
- net !RESET!/SPI_CLK11: now also RST11.2; no longer J59.28, R213.1, S23.3
- net !RESET!/SPI_CLK2: now also RST2.2; no longer J14.28, R51.1, S5.3
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Routing:
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